Commit message: rename package

File: urdf/base.urdf.xacro (robot description, xacro)
@@ -18,5 +18,5 @@
 				<origin rpy="0 0 ${M_PI if reflect == -1 else 0}" />
 				<geometry>
-					<mesh filename="package://agribot/meshes/base_block.dae" />
+					<mesh filename="package://earth_rover_description/meshes/base_block.dae" />
 				</geometry>
 				<material name="${colour}" />

File: urdf/earth_rover.urdf.xacro (robot description, xacro)
@@ -1,4 +1,4 @@
 <?xml version="1.0" encoding="UTF-8"?>
-<robot xmlns:xacro="http://www.ros.org/wiki/xacro" name="newton_agribot">
+<robot xmlns:xacro="http://www.ros.org/wiki/xacro" name="earth_rover">
 	<xacro:property name="M_PI" value="3.1415926535897931" />
 	<!-- measured mass of tyre and hub outer part: 1.238g -->
@@ -52,5 +52,5 @@
 		<visual>
 			<geometry>
-				<mesh filename="package://agribot/meshes/battery_block.dae" />
+				<mesh filename="package://earth_rover_description/meshes/battery_block.dae" />
 			</geometry>
 		</visual>

File: urdf/wheels.urdf.xacro (robot description, xacro)
@@ -26,5 +26,5 @@
 				<origin xyz="0 ${reflect*wheel_offset_y} ${wheel_offset_z}" rpy="0 0 ${M_PI if reflect == -1 else 0}"/>
 				<geometry>
-					<mesh filename="package://agribot/meshes/steering_block.dae" />
+					<mesh filename="package://earth_rover_description/meshes/steering_block.dae" />
 				</geometry>
 				<material name="silver"/>
@@ -52,5 +52,5 @@
 				</xacro:if>
 				<geometry>
-					<mesh filename="package://agribot/meshes/wheel.dae" />
+					<mesh filename="package://earth_rover_description/meshes/wheel.dae" />
 				</geometry>
 				<material name="black" />
