Commit message: [RVIZ] Added visualization of the model
Signed-off-by: Sergio A. Mart <sergio@earthrover.cc>

File: urdf/earth_rover.urdf.xacro (robot description, xacro)
@@ -18,7 +18,7 @@
 		<color rgba=".8 .8 .8 1" />
 	</material>
-	<xacro:include filename="base.urdf.xacro" />
-	<xacro:include filename="wheels.urdf.xacro" />
-	<!-- link of convenience, makes things more symmetrical -->
+  <xacro:include filename="base.urdf.xacro" />
+  <xacro:include filename="wheels.urdf.xacro" />
+  <!-- link of convenience, makes things more symmetrical -->
 	<link name="base_link"/>
 	<!-- gazebo doesn't recognise links without mass, but KDL doesn't

File: urdf/wheels.urdf.xacro (robot description, xacro)
@@ -66,26 +66,31 @@
 			<material>Gazebo/DarkGrey</material>
 		</gazebo>
-		<joint name="${name}_ankle_joint" type="revolute">
-			<parent link="${parent}" />
-			<child link="${name}_ankle" />
-			<axis xyz="0 0 1" />
-			<origin xyz="${reflect_y*ankle_offset_x} ${reflect*ankle_offset_y} -${ankle_offset_z}" />
-			<limit lower="-${angle_limit_ccw}" upper="${angle_limit_cw}" effort="7" velocity="15" /> <!-- guesses -->
-		</joint>
-		<joint name="${name}_wheel_joint" type="continuous">
-			<parent link="${name}_ankle" />
-			<child link="${name}_wheel" />
-			<axis xyz="0 1 0" />
-			<origin xyz="0 ${reflect*wheel_offset_y} ${wheel_offset_z}" />
-		</joint>
-		<!-- transmissions needed for gazebo -->
-		<transmission name="${name}_ankle_transmission" type="SimpleTransmission">
+		<!-- Steering with transmissions for gazebo -->
+    <joint name="${name}_steering_joint" type="revolute">
+      <parent link="${parent}" />
+      <child link="${name}_ankle" />
+      <axis xyz="0 0 1" />
+      <origin xyz="${reflect_y*ankle_offset_x} ${reflect*ankle_offset_y} -${ankle_offset_z}" />
+      <limit lower="-${angle_limit_ccw}" upper="${angle_limit_cw}" effort="7" velocity="15" />
+      <!-- guesses -->
+    </joint>
+    <transmission name="${name}_steering_trans" type="SimpleTransmission">
 			<type>transmission_interface/SimpleTransmission</type>
-			<actuator name="${name}_ankle_motor" />
-			<joint name="${name}_ankle_joint">
-				<hardwareInterface>EffortJointInterface</hardwareInterface>
+      <actuator name="${name}_steering_motor">
+        <hardwareInterface>PositionJointInterface</hardwareInterface>
+        <mechanicalReduction>1</mechanicalReduction>
+      </actuator>
+			<joint name="${name}_steering_joint">
+				<hardwareInterface>PositionJointInterface</hardwareInterface>
 			</joint>
 		</transmission>
-		<transmission name="${name}_wheel_transmission" type="SimpleTransmission">
+    <!-- Power wheels -->
+    <joint name="${name}_wheel_joint" type="continuous">
+      <parent link="${name}_ankle" />
+      <child link="${name}_wheel" />
+      <axis xyz="0 1 0" />
+      <origin xyz="0 ${reflect*wheel_offset_y} ${wheel_offset_z}" />
+    </joint>
+    <transmission name="${name}_wheel_transmission" type="SimpleTransmission">
 			<type>transmission_interface/SimpleTransmission</type>
 			<actuator name="${name}_wheel_motor" />

Commit message: new mass for base link

File: urdf/earth_rover.urdf.xacro (robot description, xacro)
@@ -23,10 +23,10 @@
 	<link name="base_link"/>
 	<!-- gazebo doesn't recognise links without mass, but KDL doesn't
-	     like the base link to have inertia, so we have this silly
+	     like the ba link to have inertia, so we have this silly
 	     situation of a dummy inertia link for a dummy link... -->
 	<link name="base_link_inertia">
 		<inertial>
 			<!-- mass needed for gazebo to recognise link -->
-			<mass value="0.001" />
+			<mass value="1000.00" />
 			<inertia ixx="1" iyy="1" izz="1" ixy="0" ixz="0" iyz="0" />
 		</inertial>

File: urdf/wheels.urdf.xacro (robot description, xacro)
@@ -75,4 +75,11 @@
       <!-- guesses -->
     </joint>
+	 <joint name="${name}_wheel_joint" type="continuous">
+      <parent link="${name}_ankle" />
+      <child link="${name}_wheel" />
+      <axis xyz="0 1 0" />
+      <origin xyz="0 ${reflect*wheel_offset_y} ${wheel_offset_z}" />
+    </joint>
+<!--
     <transmission name="${name}_steering_trans" type="SimpleTransmission">
 			<type>transmission_interface/SimpleTransmission</type>
@@ -85,11 +92,6 @@
 			</joint>
 		</transmission>
+-->
     <!-- Power wheels -->
-    <joint name="${name}_wheel_joint" type="continuous">
-      <parent link="${name}_ankle" />
-      <child link="${name}_wheel" />
-      <axis xyz="0 1 0" />
-      <origin xyz="0 ${reflect*wheel_offset_y} ${wheel_offset_z}" />
-    </joint>
     <transmission name="${name}_wheel_transmission" type="SimpleTransmission">
 			<type>transmission_interface/SimpleTransmission</type>
@@ -99,4 +101,11 @@
 			</joint>
 		</transmission>
+  <transmission name="${name}_steering_trans" type="SimpleTransmission">
+			<type>transmission_interface/SimpleTransmission</type>
+			<actuator name="${name}_steering_motor" />
+			<joint name="${name}_steering_joint">
+				<hardwareInterface>hardware_interface/PositionJointInterface</hardwareInterface>
+			</joint>
+		</transmission>
 	</xacro:macro>
 </robot>
